Commit message: Updated

File: control_ws/src/control_pkg/model/model.xacro (robot description, xacro)
@@ -1,68 +1,72 @@
 <?xml version="1.0"?>
-<!-- This file is part of the control_pkg package -->
-<robot name="simple robot" xmlns:xacro="http://www.ros.org/wiki/xacro" xmlns:control_pkg="http://www.control_pkg.org">
-  <xacro:include filename="$(find control_pkg)/model/parameters.xacro"/>
-  <link name="world"></link>
-  <link name="first_link">
-    <visual>
-      <origin xyz="0 0 ${s}" rpy="0 0 0"/>
-      <geometry>
-        <box size="${a} ${b} ${c}"/>
-      </geometry>
-      <material name="red"/>
-    </visual>
-    <collision>
-      <origin xyz="0 0 ${s}" rpy="0 0 0"/>
-      <geometry>
-        <box size="${a} ${b} ${c}"/>
-      </geometry>
-    </collision>
-    <xacro:inertial_body/>
-  </link>
-  <link name="second_link">
-    <visual>
-      <origin xyz="0 0 ${s}" rpy="0 0 0"/>
-      <geometry>
-        <box size="${a} ${b} ${c}"/>
-      </geometry>
-      <material name="green"/>
-    </visual>
-    <collision>
-      <origin xyz="0 0 ${s}" rpy="0 0 0"/>
-      <geometry>
-        <box size="${a} ${b} ${c}"/>
-      </geometry>
-    </collision>
-    <xacro:inertial_body/>
-  </link>
-  <joint name="fixed_joint" type="fixed">
-    <parent link="world" />
-    <child link="first_link"/>
-  </joint>
-  <joint name="first_joint" type="revolute">
-    <parent link="first_link"/>
-    <child link="second_link"/>
-    <origin xyz="0 ${b} ${q}" rpy="0 0 0"/>
-    <axis xyz="0 1 0"/>
-    <limit effort="1000" velocity="10" lower="-3.14" upper="3.14"/>
-    <dynamics damping="1.0" friction="1.0"/>
-  </joint>
-  <ros2_control name="RobotController" type="system">
-    <hardware>
-      <plugin>mock_components/GenericSystem</plugin>
-      <param name="calculate_dynamics">false</param>
-      <param name="custom_interface_with_following_offset"></param>
-      <param name="disable_commands">false</param>
-      <param name="mock_gpio_commands">false</param>
-      <param name="mock_sensor_commands">false</param>
-      <param name="position_state_following_offset">0.0</param>
-    </hardware>
-    <joint name="first_joint">
-      <command_interface name="position">
-        <param name="min">-3.14</param>
-        <param name="max">3.14</param>
-      </command_interface>
-      <state_interface name="position"/>
+<robot name="simple_robot" xmlns:xacro="http://www.ros.org/wiki/xacro">
+    <xacro:include filename="$(find control_pkg)/model/parameters.xacro"/>
+    <!-- World Link -->
+    <link name="world"></link>
+    <!-- Fixed Joint -->
+    <joint name="fixed_joint" type="fixed">
+        <parent link="world"/>
+        <child link="first_link"/>
     </joint>
-  </ros2_control>
+    <!-- First Link -->
+    <link name="first_link">
+        <visual>
+            <geometry>
+                <box size="${a} ${b} ${c}"/>
+            </geometry>
+            <origin xyz="0 0 ${s}" rpy="0 0 0"/>
+            <material name="Red"/>
+        </visual>
+        <collision>
+            <geometry>
+                <box size="${a} ${b} ${c}"/>
+            </geometry>
+            <origin xyz="0 0 ${s}" rpy="0 0 0"/>
+        </collision>
+        <xacro:inertial_body/>
+    </link>
+    <!-- Second Link -->
+    <link name="second_link">
+        <visual>
+            <geometry>
+                <box size="${a} ${b} ${c}"/>
+            </geometry>
+            <origin xyz="0 0 ${s}" rpy="0 0 0"/>
+            <material name="Green"/>
+        </visual>
+        <collision>
+            <geometry>
+                <box size="${a} ${b} ${c}"/>
+            </geometry>
+            <origin xyz="0 0 ${s}" rpy="0 0 0"/>
+        </collision>
+        <xacro:inertial_body/>
+    </link>
+    <!-- First Joint -->
+    <joint name="first_joint" type="revolute">
+        <parent link="first_link"/>
+        <child link="second_link"/>
+        <origin xyz="0 ${b} ${q}" rpy="0 0 0"/>
+        <axis xyz="0 1 0"/>
+        <limit effort="5000" velocity="10" lower="-1.571" upper="1.571"/>
+        <dynamics damping="1.0" friction="1.0"/>
+    </joint>
+    <ros2_control name="RobotController" type="system">
+        <hardware>
+            <plugin>mock_components/GenericSystem</plugin>
+            <param name="calculate_dynamics">false</param>
+            <param name="custom_interface_with_following_offset"></param>
+            <param name="disable_commands">false</param>
+            <param name="mock_gpio_commands">false</param>
+            <param name="mock_sensor_commands">false</param>
+            <param name="position_state_following_offset">0.0</param>
+        </hardware>
+        <joint name="first_joint">
+            <command_interface name="position">
+                <param name="min" value="-1.571"/>
+                <param name="max" value="1.571"/>
+            </command_interface>
+            <state_interface name="position"/>
+        </joint>
+    </ros2_control>
 </robot>

File: control_ws/src/control_pkg/model/parameters.xacro (robot description, xacro)
@@ -1,45 +1,43 @@
 <?xml version="1.0"?>
-<!-- This file is part of the control_pkg package -->
-<robot xmlns:xacro="http://www.ros.org/wiki/xacro" xmlns:control_pkg="http://www.control_pkg.org">
-  <xacro:property name="robot_name" value="control_robot"/>
-  <xacro:property name="robot_namespace" value="/control_robot"/>
-  <!-- Define robot parameters -->
-  <xacro:property name="a" value="0.1"/>
-  <xacro:property name="b" value="0.1"/>
-  <xacro:property name="c" value="0.8"/>
-  <!-- Center of mass -->
-  <xacro:property name="s" value="${c/2}"/>
-  <!-- First Joint position -->
-  <xacro:property name="q" value="${c-c/4}"/>
-  <!-- Material Density -->
-  <xacro:property name="d" value="2710"/>
-  <!-- Mass -->
-  <xacro:property name="m" value="${d * a * b * c}"/>
-  <!-- Inertia -->
-  <xacro:property name="Ixx" value="${m * (b*b + c*c)/12}"/>
-  <xacro:property name="Iyy" value="${m * (a*a + c*c)/12}"/>
-  <xacro:property name="Izz" value="${m * (a*a + b*b)/12}"/>
-  <!-- Inertial sections of the body -->
-  <xacro:macro name="inertial_body">
-    <inertial>
-      <origin xyz="0 0 ${s}" rpy="0 0 0"/>
-      <mass value="${m}"/>
-      <inertia ixx="${Ixx}" ixy="0" ixz="0" iyy="${Iyy}" iyz="0" izz="${Izz}"/>
-    </inertial>
-  </xacro:macro>
-<!-- Colors -->
-  <xacro:macro name="colors">
-    <material name="red">
-      <color rgba="1 0 0 1"/>
+<robot xmlns:xacro="http://www.ros.org/wiki/xacro">
+    <!--Link Dimensions-->
+    <xacro:property name="a" value="0.1"/>
+    <xacro:property name="b" value="0.1"/>
+    <xacro:property name="c" value="0.8"/>
+    <!--Center of Mass for first joint-->
+    <xacro:property name="s" value="${c/2}"/>
+    <!-- First Joint Displacement-->
+    <xacro:property name="q" value="${c-c/4}"/>
+    <!-- Material Density-->
+    <xacro:property name="d" value="1000"/>
+    <!-- Mass-->
+    <xacro:property name="m" value="${d*a*b*c}"/>
+    <!-- Link Moment of Inertia-->
+    <xacro:property name="Ix_body" value="${m*(b*b+c*c)/12}"/>
+    <xacro:property name="Iy_body" value="${m*(a*a+c*c)/12}"/>
+    <xacro:property name="Iz_body" value="${m*(a*a+b*b)/12}"/>
+    <!-- Inertial section of the robot body-->
+    <xacro:macro name="inertial_body">
+        <inertial>
+            <mass value="${m}"/>
+            <origin xyz="0 0 ${s}" rpy="0 0 0"/>
+            <inertia ixx="${Ix_body}" ixy="0" ixz="0" iyy="${Iy_body}" iyz="0" izz="${Iz_body}"/>
+        </inertial>
+    </xacro:macro>
+    <!-- Colors -->
+    <material name="Red">
+        <color rgba="1 0 0 1"/>
     </material>
-    <material name="green">
-      <color rgba="0 1 0 1"/>
+    <material name="Green">
+        <color rgba="0 1 0 1"/>
     </material>
-    <material name="blue">
-      <color rgba="0 0 1 1"/>
+    <material name="Blue">
+        <color rgba="0 0 1 1"/>
     </material>
-    <material name="yellow">
-      <color rgba="1 1 0 1"/>
+    <material name="Black">
+        <color rgba="0 0 0 1"/>
     </material>
-  </xacro:macro>
+    <material name="White">
+        <color rgba="1 1 1 1"/>
+    </material>
 </robot>

Commit message: Done Changes

File: control_ws/src/control_pkg/model/model.xacro (robot description, xacro)
@@ -4,9 +4,4 @@
     <!-- World Link -->
     <link name="world"></link>
-    <!-- Fixed Joint -->
-    <joint name="fixed_joint" type="fixed">
-        <parent link="world"/>
-        <child link="first_link"/>
-    </joint>
     <!-- First Link -->
     <link name="first_link">
@@ -43,4 +38,9 @@
         <xacro:inertial_body/>
     </link>
+    <!-- Fixed Joint -->
+    <joint name="fixed_joint" type="fixed">
+        <parent link="world"/>
+        <child link="first_link"/>
+    </joint>
     <!-- First Joint -->
     <joint name="first_joint" type="revolute">
